Commit message: commit according to container

File: sr_description/hand/xacro/thumb/thhub.urdf.xacro (robot description, xacro)
@@ -44,5 +44,5 @@
         <child link="${prefix}thhub" />
         <origin xyz="0 0 0.038" rpy="0 0 0" />
-        <axis xyz="${reflect} 0 0" />
+        <axis xyz="1 0 0" />
         <limit lower="${-12/180*pi}" upper="${12/180*pi}" effort="2.0" velocity="4.0" />
         <dynamics damping="0.2" />

File: sr_description/mujoco_models/urdfs/ur5_hand.urdf (robot description, URDF)
Before this commit: robot shadowhand_motor, 33 links, 32 joints
Links:
- added link ra_base
- added link ra_base_link
- added link ra_base_link_inertia, mass 4.0; collision mesh filename=package://ur_description/meshes/ur5/collision/base.stl; visual mesh filename=package://ur_description/meshes/ur5/visual/base.dae
- added link ra_flange
- added link ra_forearm_link, mass 2.275; collision mesh filename=package://ur_description/meshes/ur5/collision/forearm.stl; visual mesh filename=package://ur_description/meshes/ur5/visual/forearm.dae
- added link ra_shoulder_link, mass 3.7; collision mesh filename=package://ur_description/meshes/ur5/collision/shoulder.stl; visual mesh filename=package://ur_description/meshes/ur5/visual/shoulder.dae
- added link ra_tool0
- added link ra_upper_arm_link, mass 8.393; collision mesh filename=package://ur_description/meshes/ur5/collision/upperarm.stl; visual mesh filename=package://ur_description/meshes/ur5/visual/upperarm.dae
- added link ra_wrist_1_link, mass 1.219; collision mesh filename=package://ur_description/meshes/ur5/collision/wrist1.stl; visual mesh filename=package://ur_description/meshes/ur5/visual/wrist1.dae
- added link ra_wrist_2_link, mass 1.219; collision mesh filename=package://ur_description/meshes/ur5/collision/wrist2.stl; visual mesh filename=package://ur_description/meshes/ur5/visual/wrist2.dae
- added link ra_wrist_3_link, mass 0.1879; collision mesh filename=package://ur_description/meshes/ur5/collision/wrist3.stl; visual mesh filename=package://ur_description/meshes/ur5/visual/wrist3.dae
- link rh_forearm: geometry collision box size=0.07 0.07 0.07; collision cylinder length=0.008 radius=0.0675
Joints:
- removed joint rh_world_joint
- added joint ra_arm_to_hand: type fixed, parent ra_flange, child rh_forearm, origin xyz=0.0 0.0 0.0 rpy=1.5707963267948966 3.141592653589793 1.5707963267948966
- added joint ra_base_link-base_fixed_joint: type fixed, parent ra_base_link, child ra_base, origin xyz=0 0 0 rpy=0 0 3.141592653589793
- added joint ra_base_link-base_link_inertia: type fixed, parent ra_base_link, child ra_base_link_inertia, origin xyz=0 0 0 rpy=0 0 3.141592653589793
- added joint ra_elbow_joint: type revolute, parent ra_upper_arm_link, child ra_forearm_link, origin xyz=-0.425 0 0 rpy=0 0 0, axis 0 0 1, limit lower=-3.141592653589793 upper=3.141592653589793 effort=150.0 velocity=3.141592653589793
- added joint ra_flange-tool0: type fixed, parent ra_flange, child ra_tool0, origin xyz=0 0 0 rpy=1.5707963267948966 0 1.5707963267948966
- added joint ra_shoulder_lift_joint: type revolute, parent ra_shoulder_link, child ra_upper_arm_link, origin xyz=0 0 0 rpy=1.570796327 0 0, axis 0 0 1, limit lower=-6.283185307179586 upper=6.283185307179586 effort=150.0 velocity=3.141592653589793
- added joint ra_shoulder_pan_joint: type revolute, parent ra_base_link_inertia, child ra_shoulder_link, origin xyz=0 0 0.089159 rpy=0 0 0, axis 0 0 1, limit lower=-6.283185307179586 upper=6.283185307179586 effort=150.0 velocity=3.141592653589793
- added joint ra_wrist_1_joint: type revolute, parent ra_forearm_link, child ra_wrist_1_link, origin xyz=-0.39225 0 0.10915 rpy=0 0 0, axis 0 0 1, limit lower=-6.283185307179586 upper=6.283185307179586 effort=28.0 velocity=3.141592653589793
- added joint ra_wrist_2_joint: type revolute, parent ra_wrist_1_link, child ra_wrist_2_link, origin xyz=0 -0.09465 -1.941303950897609e-11 rpy=1.570796327 0 0, axis 0 0 1, limit lower=-6.283185307179586 upper=6.283185307179586 effort=28.0 velocity=3.141592653589793
- added joint ra_wrist_3-flange: type fixed, parent ra_wrist_3_link, child ra_flange, origin xyz=0 0 0 rpy=0 -1.5707963267948966 -1.5707963267948966
- added joint ra_wrist_3_joint: type revolute, parent ra_wrist_2_link, child ra_wrist_3_link, origin xyz=0 0.0823 -1.688001216681175e-11 rpy=1.570796326589793 3.141592653589793 3.141592653589793, axis 0 0 1, limit lower=-6.283185307179586 upper=6.283185307179586 effort=28.0 velocity=3.141592653589793
- added joint world_joint: type fixed, parent world, child ra_base_link, origin xyz=0.0 0.0 0.0 rpy=0.0 0.0 0.0
- joint rh_FFJ1: limit lower=0 upper=1.57079632679 effort=4.0 velocity=2.0 -> lower=0 upper=1.5707963267948966 effort=2 velocity=2.0
- joint rh_FFJ2: limit lower=0 upper=1.57079632679 effort=4.0 velocity=2.0 -> lower=0 upper=1.5707963267948966 effort=2 velocity=2.0
- joint rh_FFJ3: limit lower=0 upper=1.57079632679 effort=4.0 velocity=2.0 -> lower=-0.2617993877991494 upper=1.5707963267948966 effort=2 velocity=2.0
- joint rh_FFJ4: axis 0 -1.0 0 -> 0 -1 0; limit lower=-0.349065850399 upper=0.349065850399 effort=4.0 velocity=2.0 -> lower=-0.3490658503988659 upper=0.3490658503988659 effort=2 velocity=2.0
- joint rh_LFJ1: limit lower=0 upper=1.57079632679 effort=4.0 velocity=2.0 -> lower=0 upper=1.5707963267948966 effort=2 velocity=2.0
- joint rh_LFJ2: limit lower=0 upper=1.57079632679 effort=4.0 velocity=2.0 -> lower=0 upper=1.5707963267948966 effort=2 velocity=2.0
- joint rh_LFJ3: limit lower=0 upper=1.57079632679 effort=4.0 velocity=2.0 -> lower=-0.2617993877991494 upper=1.5707963267948966 effort=2 velocity=2.0
- joint rh_LFJ4: axis 0 1.0 0 -> 0 1 0; limit lower=-0.349065850399 upper=0.349065850399 effort=4.0 velocity=2.0 -> lower=-0.3490658503988659 upper=0.3490658503988659 effort=2 velocity=2.0
- joint rh_LFJ5: limit lower=0 upper=0.785398163397 effort=4.0 velocity=2.0 -> lower=0 upper=0.7853981633974483 effort=2 velocity=2.0
- joint rh_MFJ1: limit lower=0 upper=1.57079632679 effort=4.0 velocity=2.0 -> lower=0 upper=1.5707963267948966 effort=2 velocity=2.0
- joint rh_MFJ2: limit lower=0 upper=1.57079632679 effort=4.0 velocity=2.0 -> lower=0 upper=1.5707963267948966 effort=2 velocity=2.0
- joint rh_MFJ3: limit lower=0 upper=1.57079632679 effort=4.0 velocity=2.0 -> lower=-0.2617993877991494 upper=1.5707963267948966 effort=2 velocity=2.0
- joint rh_MFJ4: axis 0 -1.0 0 -> 0 -1 0; limit lower=-0.349065850399 upper=0.349065850399 effort=4.0 velocity=2.0 -> lower=-0.3490658503988659 upper=0.3490658503988659 effort=2 velocity=2.0
- joint rh_RFJ1: limit lower=0 upper=1.57079632679 effort=4.0 velocity=2.0 -> lower=0 upper=1.5707963267948966 effort=2 velocity=2.0
- joint rh_RFJ2: limit lower=0 upper=1.57079632679 effort=4.0 velocity=2.0 -> lower=0 upper=1.5707963267948966 effort=2 velocity=2.0
- joint rh_RFJ3: limit lower=0 upper=1.57079632679 effort=4.0 velocity=2.0 -> lower=-0.2617993877991494 upper=1.5707963267948966 effort=2 velocity=2.0
- joint rh_RFJ4: axis 0 1.0 0 -> 0 1 0; limit lower=-0.349065850399 upper=0.349065850399 effort=4.0 velocity=2.0 -> lower=-0.3490658503988659 upper=0.3490658503988659 effort=2 velocity=2.0
- joint rh_THJ1: limit lower=0 upper=1.57079632679 effort=4.0 velocity=4.0 -> lower=-0.2617993877991494 upper=1.5707963267948966 effort=1.0 velocity=4.0; origin xyz=0 0 0.032 rpy=0 0 -1.57079632679 -> xyz=0 0 0.032 rpy=0 0 -1.5707963267948966
- joint rh_THJ2: limit lower=-0.698131700798 upper=0.698131700798 effort=4.0 velocity=2.0 -> lower=-0.6981317007977318 upper=0.6981317007977318 effort=2.0 velocity=2.0
- joint rh_THJ3: limit lower=-0.209439510239 upper=0.209439510239 effort=4.0 velocity=4.0 -> lower=-0.20943951023931953 upper=0.20943951023931953 effort=2.0 velocity=4.0
- joint rh_THJ4: axis 1.0 0 0 -> 1 0 0; limit lower=0.0 upper=1.2217304764 effort=4.0 velocity=4.0 -> lower=0.0 upper=1.2217304763960306 effort=3 velocity=4.0
- joint rh_THJ5: axis 0 0 -1.0 -> 0 0 -1; limit lower=-1.0471975512 upper=1.0471975512 effort=4.0 velocity=4.0 -> lower=-1.0471975511965976 upper=1.0471975511965976 effort=5.0 velocity=4.0; origin xyz=0.034 -0.0085 0.029 rpy=0 0.785398163397 0.0 -> xyz=0.034 -0.00858 0.029 rpy=0 0.7853981633974483 0.0
- joint rh_WRJ1: limit lower=-0.698131700798 upper=0.488692190558 effort=5.0 velocity=2.0 -> lower=-0.6981317007977318 upper=0.4886921905584123 effort=30 velocity=2.0
- joint rh_WRJ2: axis 0 1.0 0 -> 0 1 0; limit lower=-0.523598775598 upper=0.174532925199 effort=10.0 velocity=2.0 -> lower=-0.5235987755982988 upper=0.17453292519943295 effort=10 velocity=2.0; origin xyz=0 -0.010 0.213 rpy=0 0 0 -> xyz=0 -0.010 0.21301 rpy=0 0 0

File: sr_description/robots/sr_hand.urdf.xacro (robot description, xacro)
@@ -16,5 +16,5 @@
   <xacro:arg name="palm_sensor" default="none"/>
   <xacro:arg name="mounting_plate" default="false"/>
-  <link name="world" />
+  <link name="world"/>
   <xacro:if value="${'$(arg side)' == 'right'}">
     <joint name="rh_world_joint" type="fixed">
